Commit message: x

File: src/lab3/dynamic.urdf (robot description, URDF)
Before this commit: robot visual, 6 links, 5 joints
Links:
- link cylinder_3: geometry visual cylinder length=0.3 radius=0.1
Joints:
- joint cylinder_1_cylinder_2: axis 0 -1 0 -> 0 1.0 0; origin xyz=0 0 1.0 -> xyz=0 0 1.0 rpy=0 0 0
