Commit message: x

File: src/lab4/dynamic.urdf (robot description, URDF)
Before this commit: robot visual, 6 links, 5 joints
Joints:
- joint cylinder_1_cylinder_2: limit (none) -> lower=-1.570 upper=1.570 effort=1000.0 velocity=1; type continuous -> revolute
- joint cylinder_2_cylinder_3: limit (none) -> lower=-1.570 upper=1.570 effort=1000.0 velocity=1; type continuous -> revolute

Commit message: lab5 added without params

File: src/lab4/dynamic.urdf (robot description, URDF)
Before this commit: robot visual, 6 links, 5 joints
Joints:
- joint base_link_cylinder_1: origin xyz=0 0 0.0 -> xyz=0 0 0.0 rpy=0 0 3.14159

Commit message: x

File: src/lab4/dynamic.urdf (robot description, URDF)
Before this commit: robot visual, 6 links, 5 joints
Links:
- link cylinder_1: geometry visual cylinder length=1.0 radius=0.2
- link cylinder_2: geometry visual cylinder length=1.0 radius=0.2
